Commit message: Fix Gazebo Harmonic plugin names, ParameterFile, and camera_link collision

File: mini_pupper_description/urdf/mini_pupper/mini_pupper_description.urdf.xacro (robot description, xacro)
@@ -1488,5 +1488,5 @@
   <ros2_control name="GazeboSystem" type="system">
     <hardware>
-      <plugin>gz_ros2_control/GazeboSystem</plugin>
+      <plugin>gz_ros2_control/GazeboSimSystem</plugin>
     </hardware>
     <joint name="base_lf1">
@@ -1777,5 +1777,5 @@
   </gazebo>
   <gazebo>
-    <plugin filename="gz_ros2_control.so" name="gazebo_ros2_control">
+    <plugin filename="gz_ros2_control-system" name="gz_ros2_control::GazeboSimROS2ControlPlugin">
       <parameters>$(find mini_pupper_description)/config/ros_control/mini_pupper_controller.yaml</parameters>
     </plugin>

File: mini_pupper_description/urdf/mini_pupper_2/mini_pupper_description.urdf.xacro (robot description, xacro)
@@ -837,5 +837,5 @@
   <ros2_control name="GazeboSystem" type="system">
     <hardware>
-      <plugin>gz_ros2_control/GazeboSystem</plugin>
+      <plugin>gz_ros2_control/GazeboSimSystem</plugin>
     </hardware>
     <joint name="base_lf1">
@@ -1137,5 +1137,5 @@
   </gazebo>
   <gazebo>
-    <plugin filename="gz_ros2_control.so" name="gazebo_ros2_control">
+    <plugin filename="gz_ros2_control-system" name="gz_ros2_control::GazeboSimROS2ControlPlugin">
       <parameters>$(find mini_pupper_description)/config/ros_control/mini_pupper_2_controller.yaml</parameters>
     </plugin>
@@ -1177,4 +1177,11 @@
       </material>
     </visual>
+    <collision>
+      <geometry>
+        <box>
+          <size>0.02 0.02 0.02</size>
+        </box>
+      </geometry>
+    </collision>
   </link>
   <joint name="bodyfront_camera_joint" type="fixed">
