Commit message: Remove gz_ros2_base.so plugin and fix camera_link box syntax

File: mini_pupper_description/urdf/mini_pupper_2/mini_pupper_description.urdf.xacro (robot description, xacro)
@@ -1124,17 +1124,4 @@
   </gazebo>
   <gazebo>
-    <plugin filename="gz_ros2_base.so" name="p3d_base_controller">
-      <ros>
-        <remapping>odom:=odom/ground_truth</remapping>
-      </ros>
-      <body_name>base_link</body_name>
-      <frame_name>world</frame_name>
-      <update_rate>10.0</update_rate>
-      <xyz_offset>0 0 0</xyz_offset>
-      <rpy_offset>0 0 0</rpy_offset>
-      <gaussian_noise>0.01</gaussian_noise>
-    </plugin>
-  </gazebo>
-  <gazebo>
     <plugin filename="gz_ros2_control-system" name="gz_ros2_control::GazeboSimROS2ControlPlugin">
       <parameters>$(find mini_pupper_description)/config/ros_control/mini_pupper_2_controller.yaml</parameters>
@@ -1168,7 +1155,5 @@
     <visual>
       <geometry>
-        <box>
-          <size>0.02 0.02 0.02</size>
-        </box>
+        <box size="0.02 0.02 0.02"/>
       </geometry>
       <material>
@@ -1179,7 +1164,5 @@
     <collision>
       <geometry>
-        <box>
-          <size>0.02 0.02 0.02</size>
-        </box>
+        <box size="0.02 0.02 0.02"/>
       </geometry>
     </collision>

Commit message: Revert camera_link collision fix - not required for Jazzy migration

File: mini_pupper_description/urdf/mini_pupper_2/mini_pupper_description.urdf.xacro (robot description, xacro)
@@ -1149,9 +1149,4 @@
       </material>
     </visual>
-    <collision>
-      <geometry>
-        <box size="0.02 0.02 0.02"/>
-      </geometry>
-    </collision>
   </link>
   <joint name="bodyfront_camera_joint" type="fixed">

Commit message: Fix camera_link material missing name attribute

File: mini_pupper_description/urdf/mini_pupper_2/mini_pupper_description.urdf.xacro (robot description, xacro)
@@ -1144,5 +1144,5 @@
         <box size="0.02 0.02 0.02"/>
       </geometry>
-      <material>
+      <material name="blue">
         <ambient>0 0 1 1</ambient>
         <diffuse>0 0 1 1</diffuse>
